Commit message: update urdf

File: urdf/gazebo_control.xacro (robot description, xacro)
@@ -36,4 +36,7 @@
         <mu1>1.0</mu1>
         <mu2>1.0</mu2>
+        <!--kp>10000000.0</kp-->
+        <kd>1.0</kd>
+        <minDepth>0.005</minDepth> <fdir1>1 0 0</fdir1>
     </gazebo>
     <gazebo reference="right_wheel">
@@ -41,10 +44,16 @@
         <mu1>1.0</mu1>
         <mu2>1.0</mu2>
+        <!--kp>10000000.0</kp-->
+        <kd>1.0</kd>
+        <minDepth>0.005</minDepth> <fdir1>1 0 0</fdir1>
     </gazebo>
     <gazebo reference="caster_wheel">
         <material>Gazebo/Black</material>
-        <mu1>0.001</mu1> <mu2>0.001</mu2>
+        <mu1>0.001</mu1>
+        <mu2>0.001</mu2>
+        <minDepth>0.005</minDepth> <fdir1>1 0 0</fdir1>
     </gazebo>
     <gazebo reference="laser_frame">
+        <material>Gazebo/Black</material>
         <sensor name="lidar" type="ray">
             <pose>0 0 0 0 0 0</pose>
@@ -61,5 +70,5 @@
                 </scan>
                 <range>
-                    <min>0.12</min> <max>3.5</max>
+                    <min>0.20</min> <max>3.5</max>
                 </range>
             </ray>

File: urdf/mobile_robot.urdf.xacro (robot description, xacro)
@@ -11,7 +11,13 @@
     <xacro:property name="wheel_mass" value="1.5"/>
     <xacro:property name="wheel_offset_y" value="${(chassis_width / 2) + (wheel_width / 2)}"/>
-    <xacro:property name="caster_radius" value="0.06"/>
+    <xacro:property name="caster_radius" value="0.10499"/>
     <xacro:property name="caster_mass" value="0.5"/>
-    <link name="base_link"></link>
+    <link name="base_link">
+        <inertial>
+            <mass value="0.1"/>
+            <origin xyz="0 0 0" rpy="0 0 0"/>
+            <inertia ixx="0.001" ixy="0.0" ixz="0.0" iyy="0.001" iyz="0.0" izz="0.001"/>
+        </inertial>
+    </link>
     <link name="base_footprint"/>
     <joint name="base_joint" type="fixed">
@@ -34,5 +40,5 @@
         </visual>
         <collision>
-            <origin xyz="0 0 ${chassis_height/2}" rpy="0 0 0"/>
+            <origin xyz="${chassis_width/3.5} 0 ${chassis_height/2}" rpy="0 0 0"/>
             <geometry>
                 <box size="${chassis_length} ${chassis_width} ${chassis_height}"/>
@@ -40,5 +46,5 @@
         </collision>
         <xacro:inertial_box mass="${chassis_mass}" x="${chassis_length}" y="${chassis_width}" z="${chassis_height}">
-            <origin xyz="0 0 ${chassis_height/2}" rpy="0 0 0"/>
+            <origin xyz="0.15 0 0.1" rpy="0 0 0"/>
         </xacro:inertial_box>
     </link>
@@ -46,6 +52,6 @@
         <parent link="base_link"/>
         <child link="left_wheel"/>
-        <origin xyz="0 ${wheel_offset_y} 0" rpy="0 -${pi/2} 0"/>
-        <axis xyz="0 0 1"/>
+        <origin xyz="0 ${wheel_offset_y} 0" rpy="0 0 0"/>
+        <axis xyz="0 1 0"/>
     </joint>
     <link name="left_wheel">
@@ -58,4 +64,5 @@
         </visual>
         <collision>
+            <origin xyz="0 0 0" rpy="${pi/2} 0 0"/>
             <geometry>
                 <cylinder radius="${wheel_radius}" length="${wheel_width}"/>
@@ -63,5 +70,5 @@
         </collision>
         <xacro:inertial_cylinder mass="${wheel_mass}" length="${wheel_width}" radius="${wheel_radius}">
-            <origin xyz="0 0 0" rpy="0 0 0"/>
+            <origin xyz="0 0 0" rpy="${pi/2} 0 0"/>
         </xacro:inertial_cylinder>
     </link>
@@ -69,6 +76,6 @@
         <parent link="base_link"/>
         <child link="right_wheel"/>
-        <origin xyz="0 -${wheel_offset_y} 0" rpy="0 ${pi/2} 0"/>
-        <axis xyz="0 0 -1"/>
+        <origin xyz="0 -${wheel_offset_y} 0" rpy="0 0 0"/>
+        <axis xyz="0 1 0"/>
     </joint>
     <link name="right_wheel">
@@ -81,4 +88,5 @@
         </visual>
         <collision>
+            <origin xyz="0 0 0" rpy="${pi/2} 0 0"/>
             <geometry>
                 <cylinder radius="${wheel_radius}" length="${wheel_width}"/>
@@ -86,5 +94,5 @@
         </collision>
         <xacro:inertial_cylinder mass="${wheel_mass}" length="${wheel_width}" radius="${wheel_radius}">
-            <origin xyz="0 0 0" rpy="0 0 0"/>
+            <origin xyz="0 0 0" rpy="${pi/2} 0 0"/>
         </xacro:inertial_cylinder>
     </link>
@@ -92,5 +100,5 @@
         <parent link="chassis"/>
         <child link="caster_wheel"/>
-        <origin xyz="-0.3 0 -${chassis_height/2}" rpy="0 0 0"/>
+        <origin xyz="0.248 0 0.023" rpy="0 0 0"/>
     </joint>
     <link name="caster_wheel">
@@ -103,7 +111,7 @@
         </visual>
         <collision>
-            <origin xyz="0 0 ${-caster_radius/2}" rpy="0 0 0"/>
+            <origin xyz="0 0 ${-(caster_radius/2)}" rpy="0 0 0"/>
             <geometry>
-                <sphere radius="${caster_radius}"/>
+                <sphere radius="${caster_radius/2}"/>
             </geometry>
         </collision>
@@ -115,5 +123,5 @@
         <parent link="chassis"/>
         <child link="laser_frame"/>
-        <origin xyz="0 0 ${chassis_height}" rpy="0 0 0"/>
+        <origin xyz="${chassis_width/2} 0 ${chassis_height/4 - 0.02}" rpy="0 0 0"/>
     </joint>
     <link name="laser_frame">

Commit message: add imu to urdf

File: urdf/gazebo_control.xacro (robot description, xacro)
@@ -82,3 +82,32 @@
         </sensor>
     </gazebo>
+    <gazebo reference="imu_link">
+        <gravity>true</gravity>
+        <sensor name="imu_sensor" type="imu">
+            <always_on>true</always_on>
+            <update_rate>100</update_rate>
+            <visualize>true</visualize>
+            <topic>__default_topic__</topic>
+            <imu>
+                <angular_velocity>
+                    <x><noise type="gaussian"><mean>0.0</mean><stddev>2e-4</stddev></noise></x>
+                    <y><noise type="gaussian"><mean>0.0</mean><stddev>2e-4</stddev></noise></y>
+                    <z><noise type="gaussian"><mean>0.0</mean><stddev>2e-4</stddev></noise></z>
+                </angular_velocity>
+                <linear_acceleration>
+                    <x><noise type="gaussian"><mean>0.0</mean><stddev>1.7e-2</stddev></noise></x>
+                    <y><noise type="gaussian"><mean>0.0</mean><stddev>1.7e-2</stddev></noise></y>
+                    <z><noise type="gaussian"><mean>0.0</mean><stddev>1.7e-2</stddev></noise></z>
+                </linear_acceleration>
+            </imu>
+            <plugin filename="libgazebo_ros_imu_sensor.so" name="imu_plugin">
+                <ros>
+                    <remapping>~/out:=/imu</remapping>
+                </ros>
+                <frame_name>imu_link</frame_name>
+                <initial_orientation_as_reference>false</initial_orientation_as_reference>
+            </plugin>
+            <pose>0 0 0 0 0 0</pose>
+        </sensor>
+    </gazebo>
 </robot>

File: urdf/mobile_robot.urdf.xacro (robot description, xacro)
@@ -141,3 +141,23 @@
         </xacro:inertial_cylinder>
     </link>
+    <joint name="imu_joint" type="fixed">
+        <parent link="chassis"/>
+        <child link="imu_link"/>
+        <origin xyz="0 0 ${chassis_height/4}" rpy="0 0 0"/>
+    </joint>
+    <link name="imu_link">
+        <visual>
+            <geometry>
+                <box size="0.02 0.02 0.01"/>
+            </geometry>
+            <material name="blue"/> </visual>
+        <collision>
+            <geometry>
+                <box size="0.02 0.02 0.01"/>
+            </geometry>
+        </collision>
+        <xacro:inertial_box mass="0.01" x="0.02" y="0.02" z="0.01">
+            <origin xyz="0 0 0" rpy="0 0 0"/>
+        </xacro:inertial_box>
+    </link>
 </robot>

Commit message: Update laser sensor parameters and replace chassis geometry with mesh model

File: urdf/gazebo_control.xacro (robot description, xacro)
@@ -70,5 +70,6 @@
                 </scan>
                 <range>
-                    <min>0.20</min> <max>3.5</max>
+                    <min>0.05</min> <max>30.0</max>
+                    <resolution>0.01</resolution>
                 </range>
             </ray>

File: urdf/mobile_robot.urdf.xacro (robot description, xacro)
@@ -40,7 +40,6 @@
         </visual>
         <collision>
-            <origin xyz="${chassis_width/3.5} 0 ${chassis_height/2}" rpy="0 0 0"/>
             <geometry>
-                <box size="${chassis_length} ${chassis_width} ${chassis_height}"/>
+                <mesh filename="package://mobile_robot/meshes/Model.stl" scale="0.01 0.01 0.01"/>
             </geometry>
         </collision>

Commit message: Add laser filter configuration, joystick launch file, and update URDF properties
- Introduced laser filter parameters in `laser_filter.yaml`.
- Added joystick launch file for teleoperation.
- Updated `sim_slam.launch.py` to include laser scan filtering.
- Modified URDF files to adjust wheel dimensions and removed unused materials.
- Enhanced robot teleoperation script with new key mappings.

File: urdf/gazebo_control.xacro (robot description, xacro)
@@ -10,11 +10,11 @@
             <left_joint>left_wheel_joint</left_joint>
             <right_joint>right_wheel_joint</right_joint>
-            <wheel_separation>0.45</wheel_separation>
-            <wheel_diameter>0.165</wheel_diameter>
+            <wheel_separation>0.42109</wheel_separation>
+            <wheel_diameter>0.1651</wheel_diameter>
             <max_wheel_torque>20</max_wheel_torque>
             <max_wheel_acceleration>1.0</max_wheel_acceleration>
             <publish_odom>true</publish_odom>
             <publish_odom_tf>true</publish_odom_tf>
-            <publish_wheel_tf>true</publish_wheel_tf>
+            <publish_wheel_tf>false</publish_wheel_tf>
             <odometry_frame>odom</odometry_frame>
             <robot_base_frame>base_footprint</robot_base_frame>
@@ -70,5 +70,5 @@
                 </scan>
                 <range>
-                    <min>0.05</min> <max>30.0</max>
+                    <min>0.06</min> <max>30.0</max>
                     <resolution>0.01</resolution>
                 </range>
@@ -76,5 +76,5 @@
             <plugin name="laser_controller" filename="libgazebo_ros_ray_sensor.so">
                 <ros>
-                    <argument>~/out:=scan</argument>
+                    <remapping>~/out:=scan</remapping>
                 </ros>
                 <output_type>sensor_msgs/LaserScan</output_type>

File: urdf/mobile_robot.urdf.xacro (robot description, xacro)
@@ -1,9 +1,49 @@
 <?xml version="1.0"?>
 <robot xmlns:xacro="http://www.ros.org/wiki/xacro" name="mobile_robot">
-    <xacro:include filename="materials.xacro" />
+    <!-- ==================== MATERIALS & MACROS ==================== -->
+    <material name="white">
+        <color rgba="1 1 1 1"/>
+    </material>
+    <material name="orange">
+        <color rgba="1 0.3 0.1 1"/>
+    </material>
+    <material name="blue">
+        <color rgba="0.2 0.2 1 1"/>
+    </material>
+    <material name="black">
+        <color rgba="0 0 0 1"/>
+    </material>
+    <xacro:macro name="inertial_box" params="mass x y z *origin">
+        <inertial>
+            <xacro:insert_block name="origin"/>
+            <mass value="${mass}" />
+            <inertia ixx="${(1/12) * mass * (y*y+z*z)}" ixy="0.0" ixz="0.0"
+                     iyy="${(1/12) * mass * (x*x+z*z)}" iyz="0.0"
+                     izz="${(1/12) * mass * (x*x+y*y)}" />
+        </inertial>
+    </xacro:macro>
+    <xacro:macro name="inertial_cylinder" params="mass length radius *origin">
+        <inertial>
+            <xacro:insert_block name="origin"/>
+            <mass value="${mass}" />
+            <inertia ixx="${(1/12) * mass * (3*radius*radius + length*length)}" ixy="0.0" ixz="0.0"
+                     iyy="${(1/12) * mass * (3*radius*radius + length*length)}" iyz="0.0"
+                     izz="${(1/2) * mass * (radius*radius)}" />
+        </inertial>
+    </xacro:macro>
+    <xacro:macro name="inertial_sphere" params="mass radius *origin">
+        <inertial>
+            <xacro:insert_block name="origin"/>
+            <mass value="${mass}" />
+            <inertia ixx="${(2/5) * mass * (radius*radius)}" ixy="0.0" ixz="0.0"
+                     iyy="${(2/5) * mass * (radius*radius)}" iyz="0.0"
+                     izz="${(2/5) * mass * (radius*radius)}" />
+        </inertial>
+    </xacro:macro>
     <xacro:include filename="gazebo_control.xacro" />
+    <!-- ==================== PROPERTIES ==================== -->
     <xacro:property name="chassis_length" value="0.38"/>
     <xacro:property name="chassis_width" value="0.38"/>
-    <xacro:property name="chassis_height" value="01.28577"/>
+    <xacro:property name="chassis_height" value="1.28577"/>
     <xacro:property name="chassis_mass" value="25.0"/>
     <xacro:property name="wheel_radius" value="0.08255"/>
@@ -13,4 +53,5 @@
     <xacro:property name="caster_radius" value="0.10499"/>
     <xacro:property name="caster_mass" value="0.5"/>
+    <!-- ==================== LINKS & JOINTS ==================== -->
     <link name="base_link">
         <inertial>
@@ -143,5 +184,5 @@
         <parent link="chassis"/>
         <child link="imu_link"/>
-        <origin xyz="0 0 ${chassis_height/4}" rpy="0 0 0"/>
+        <origin xyz="0 0 ${chassis_height/4 - 0.04}" rpy="0 0 0"/>
     </joint>
     <link name="imu_link">
