Commit message: update mobile_robot.urdf

File: urdf/mobile_robot.urdf.xacro (robot description, xacro)
@@ -46,5 +46,5 @@
         </collision>
         <xacro:inertial_box mass="${chassis_mass}" x="${chassis_length}" y="${chassis_width}" z="${chassis_height}">
-            <origin xyz="0.15 0 0.1" rpy="0 0 0"/>
+            <origin xyz="0.15 0 0.3" rpy="0 0 0"/>
         </xacro:inertial_box>
     </link>

Commit message: Update RViz configuration and remove obsolete URDF file for improved robot simulation

File: urdf/mobile_robot.urdf.xacro (robot description, xacro)
@@ -163,5 +163,5 @@
         <parent link="chassis"/>
         <child link="laser_frame"/>
-        <origin xyz="${chassis_width/2} 0 ${chassis_height/4 - 0.02}" rpy="0 0 0"/>
+        <origin xyz="0.248 0 ${chassis_height/18}" rpy="0 0 0"/>
     </joint>
     <link name="laser_frame">
