Commit message: Add test_dropoff world with various obstacles and platforms for robot navigation testing

File: urdf/mobile_robot_v2.urdf.xacro (robot description, xacro)
@@ -41,5 +41,5 @@
         </inertial>
     </xacro:macro>
-    <xacro:include filename="gazebo_control.xacro" />
+    <xacro:include filename="gazebo_control_v2.xacro" />
     <!-- ==================== PROPERTIES ==================== -->
     <xacro:property name="chassis_length" value="0.38"/>
@@ -74,13 +74,16 @@
     <link name="chassis">
         <visual>
-            <origin xyz="0 0 0" rpy="0 0 0"/>
-            <geometry>
-                <mesh filename="package://mobile_robot/meshes/Model.stl" scale="0.01 0.01 0.01"/>
+            <!-- <origin xyz="0.03 0 0.05" rpy="0 0 0"/> -->
+            <origin xyz="0 0 0" rpy="0 0 0"/>
+            <geometry>
+                <mesh filename="package://mobile_robot/meshes/Model_v2.stl" scale="0.001 0.001 0.001"/>
             </geometry>
             <material name="white"/>
         </visual>
         <collision>
-            <geometry>
-                <mesh filename="package://mobile_robot/meshes/Model.stl" scale="0.01 0.01 0.01"/>
+            <!-- <origin xyz="0.03 0 0.05" rpy="0 0 0"/> -->
+            <origin xyz="0 0 0" rpy="0 0 0"/>
+            <geometry>
+                <mesh filename="package://mobile_robot/meshes/Model_v2.stl" scale="0.001 0.001 0.001"/>
             </geometry>
         </collision>
@@ -163,10 +166,11 @@
         <parent link="chassis"/>
         <child link="laser_frame"/>
-        <origin xyz="0.248 0 ${chassis_height/18}" rpy="0 0 0"/>
+        <origin xyz="0.257 0 0.075" rpy="0 0 0"/>
     </joint>
     <link name="laser_frame">
         <visual>
-            <origin xyz="-0.52 0.04 -0.02" rpy="0 0 -1.570796"/>
-            <geometry>
+            <origin xyz="0 0 0" rpy="0 0 0"/>
+            <geometry>
+                <!-- <cylinder length="0.04" radius="0.038"/> -->
                 <mesh filename="package://mobile_robot/meshes/RPLiDAR_s2.stl" scale="0.001 0.001 0.001"/>
             </geometry>
@@ -174,9 +178,11 @@
         </visual>
         <collision>
-            <geometry>
+            <origin xyz="0 0 0" rpy="0 0 0"/>
+            <geometry>
+                <!-- <cylinder length="0.04" radius="0.038"/> -->
                 <mesh filename="package://mobile_robot/meshes/RPLiDAR_s2.stl" scale="0.001 0.001 0.001"/>
             </geometry>
         </collision>
-        <xacro:inertial_cylinder mass="0.1" length="0.04" radius="0.05">
+        <xacro:inertial_cylinder mass="0.1" length="0.04" radius="0.038">
             <origin xyz="0 0 0" rpy="0 0 0"/>
         </xacro:inertial_cylinder>
@@ -202,3 +208,53 @@
         </xacro:inertial_box>
     </link>
+    <xacro:macro name="ultrasonic_link" params="name">
+        <link name="${name}_link">
+            <visual>
+                <geometry><box size="0.015 0.04 0.02"/></geometry>
+                <material name="blue"/>
+            </visual>
+            <!-- <collision>
+                <geometry><box size="0.015 0.04 0.02"/></geometry>
+            </collision> -->
+            <xacro:inertial_box mass="0.01" x="0.02" y="0.04" z="0.015">
+                <origin xyz="0 0 0" rpy="0 0 0"/>
+            </xacro:inertial_box>
+        </link>
+    </xacro:macro>
+    <joint name="us_top_left_joint" type="fixed">
+        <parent link="chassis"/>
+        <child link="us_top_left_link"/>
+        <origin xyz="0.35 0.17 0.49" rpy="0 0.4363 0"/>
+    </joint>
+    <xacro:ultrasonic_link name="us_top_left"/>
+    <joint name="us_top_right_joint" type="fixed">
+        <parent link="chassis"/>
+        <child link="us_top_right_link"/>
+        <origin xyz="0.35 -0.17 0.49" rpy="0 0.4363 0"/>
+    </joint>
+    <xacro:ultrasonic_link name="us_top_right"/>
+    <joint name="us_mid_left_joint" type="fixed">
+        <parent link="chassis"/>
+        <child link="us_mid_left_link"/>
+        <origin xyz="0.35 0.17 0.257" rpy="0 -0.2618 0"/>
+    </joint>
+    <xacro:ultrasonic_link name="us_mid_left"/>
+    <joint name="us_mid_right_joint" type="fixed">
+        <parent link="chassis"/>
+        <child link="us_mid_right_link"/>
+        <origin xyz="0.35 -0.17 0.257" rpy="0 -0.2618 0"/>
+    </joint>
+    <xacro:ultrasonic_link name="us_mid_right"/>
+    <joint name="us_bot_left_joint" type="fixed">
+        <parent link="chassis"/>
+        <child link="us_bot_left_link"/>
+        <origin xyz="0.35 0.17 0.03" rpy="0 0.2618 0"/>
+    </joint>
+    <xacro:ultrasonic_link name="us_bot_left"/>
+    <joint name="us_bot_right_joint" type="fixed">
+        <parent link="chassis"/>
+        <child link="us_bot_right_link"/>
+        <origin xyz="0.35 -0.17 0.03" rpy="0 0.2618 0"/>
+    </joint>
+    <xacro:ultrasonic_link name="us_bot_right"/>
 </robot>
