Commit message: Refactor code structure for improved readability and maintainability

File: urdf/gazebo_control_v2.xacro (robot description, xacro)
@@ -157,9 +157,11 @@
         </gazebo>
     </xacro:macro>
-    <xacro:gazebo_ultrasonic name="us_top_left"   max_range="4.0" fov="0.2618"/>
-    <xacro:gazebo_ultrasonic name="us_top_right"  max_range="4.0" fov="0.2618"/>
-    <xacro:gazebo_ultrasonic name="us_mid_left"   max_range="4.0" fov="0.2618"/>
-    <xacro:gazebo_ultrasonic name="us_mid_right"  max_range="4.0" fov="0.2618"/>
-    <xacro:gazebo_ultrasonic name="us_bot_left"   max_range="0.5" fov="0.1745"/>
-    <xacro:gazebo_ultrasonic name="us_bot_right"  max_range="0.5" fov="0.1745"/>
+    <xacro:gazebo_ultrasonic name="us_top_left"   max_range="2.5" fov="0.2618"/>
+    <xacro:gazebo_ultrasonic name="us_top_right"  max_range="2.5" fov="0.2618"/>
+    <xacro:gazebo_ultrasonic name="us_mid_1_left"   max_range="2.5" fov="0.2618"/>
+    <xacro:gazebo_ultrasonic name="us_mid_1_right"  max_range="2.5" fov="0.2618"/>
+    <xacro:gazebo_ultrasonic name="us_mid_2_left"   max_range="2.5" fov="0.2618"/>
+    <xacro:gazebo_ultrasonic name="us_mid_2_right"  max_range="2.5" fov="0.2618"/>
+    <xacro:gazebo_ultrasonic name="us_bot_left"   max_range="2.5" fov="0.2618"/>
+    <xacro:gazebo_ultrasonic name="us_bot_right"  max_range="2.5" fov="0.2618"/>
 </robot>

File: urdf/mobile_robot_v2.urdf.xacro (robot description, xacro)
@@ -211,11 +211,11 @@
         <link name="${name}_link">
             <visual>
-                <geometry><box size="0.015 0.04 0.02"/></geometry>
+                <geometry><box size="0.015 0.02 0.04"/></geometry>
                 <material name="blue"/>
             </visual>
-            <!-- <collision>
-                <geometry><box size="0.015 0.04 0.02"/></geometry>
-            </collision> -->
-            <xacro:inertial_box mass="0.01" x="0.02" y="0.04" z="0.015">
+            <collision>
+                <geometry><box size="0.015 0.02 0.04"/></geometry>
+            </collision>
+            <xacro:inertial_box mass="0.01" x="0.015" y="0.02" z="0.04">
                 <origin xyz="0 0 0" rpy="0 0 0"/>
             </xacro:inertial_box>
@@ -225,5 +225,5 @@
         <parent link="chassis"/>
         <child link="us_top_left_link"/>
-        <origin xyz="0.35 0.17 0.49" rpy="0 0.4363 0"/>
+        <origin xyz="0.35 0.17 0.48" rpy="0 0 0"/>
     </joint>
     <xacro:ultrasonic_link name="us_top_left"/>
@@ -231,23 +231,35 @@
         <parent link="chassis"/>
         <child link="us_top_right_link"/>
-        <origin xyz="0.35 -0.17 0.49" rpy="0 0.4363 0"/>
+        <origin xyz="0.35 -0.17 0.48" rpy="0 0 0"/>
     </joint>
     <xacro:ultrasonic_link name="us_top_right"/>
-    <joint name="us_mid_left_joint" type="fixed">
-        <parent link="chassis"/>
-        <child link="us_mid_left_link"/>
-        <origin xyz="0.35 0.17 0.257" rpy="0 -0.2618 0"/>
-    </joint>
-    <xacro:ultrasonic_link name="us_mid_left"/>
-    <joint name="us_mid_right_joint" type="fixed">
-        <parent link="chassis"/>
-        <child link="us_mid_right_link"/>
-        <origin xyz="0.35 -0.17 0.257" rpy="0 -0.2618 0"/>
-    </joint>
-    <xacro:ultrasonic_link name="us_mid_right"/>
+    <joint name="us_mid_1_left_joint" type="fixed">
+        <parent link="chassis"/>
+        <child link="us_mid_1_left_link"/>
+        <origin xyz="0.35 0.17 0.36" rpy="0 0 0"/>
+    </joint>
+    <xacro:ultrasonic_link name="us_mid_1_left"/>
+    <joint name="us_mid_1_right_joint" type="fixed">
+        <parent link="chassis"/>
+        <child link="us_mid_1_right_link"/>
+        <origin xyz="0.35 -0.17 0.36" rpy="0 0 0"/>
+    </joint>
+    <xacro:ultrasonic_link name="us_mid_1_right"/>
+    <joint name="us_mid_2_left_joint" type="fixed">
+        <parent link="chassis"/>
+        <child link="us_mid_2_left_link"/>
+        <origin xyz="0.35 0.17 0.24" rpy="0 0 0"/>
+    </joint>
+    <xacro:ultrasonic_link name="us_mid_2_left"/>
+    <joint name="us_mid_2_right_joint" type="fixed">
+        <parent link="chassis"/>
+        <child link="us_mid_2_right_link"/>
+        <origin xyz="0.35 -0.17 0.24" rpy="0 0 0"/>
+    </joint>
+    <xacro:ultrasonic_link name="us_mid_2_right"/>
     <joint name="us_bot_left_joint" type="fixed">
         <parent link="chassis"/>
         <child link="us_bot_left_link"/>
-        <origin xyz="0.35 0.17 0.03" rpy="0 0.2618 0"/>
+        <origin xyz="0.35 0.17 0.12" rpy="0 0 0"/>
     </joint>
     <xacro:ultrasonic_link name="us_bot_left"/>
@@ -255,5 +267,5 @@
         <parent link="chassis"/>
         <child link="us_bot_right_link"/>
-        <origin xyz="0.35 -0.17 0.03" rpy="0 0.2618 0"/>
+        <origin xyz="0.35 -0.17 0.12" rpy="0 0 0"/>
     </joint>
     <xacro:ultrasonic_link name="us_bot_right"/>
