Commit message: Refactor ultrasonic fusion node and update URDF models
- Updated range parameters in ultrasonic_fusion_node.py to improve sensor accuracy.
- Adjusted obstacle detection threshold in ultrasonic_fusion_node_v2.py for better responsiveness.
- Introduced ultrasonic_fusion_node_v3.py with enhanced filtering and hard stop logic.
- Modified URDF files to reflect changes in ultrasonic sensor configurations and dimensions.
- Updated gazebo_control_x.xacro files to align with new sensor ranges and configurations.
- Corrected dimensions and orientations of ultrasonic sensors in mobile_robot URDF files.

File: urdf/gazebo_control_v3.xacro (robot description, xacro)
@@ -124,9 +124,9 @@
                             <samples>5</samples>
                             <resolution>1</resolution>
-                            <min_angle>${-fov/2}</min_angle>
-                            <max_angle>${fov/2}</max_angle>
+                            <min_angle>0</min_angle>
+                            <max_angle>0</max_angle>
                         </horizontal>
                         <vertical>
-                            <samples>5</samples>
+                            <samples>10</samples>
                             <resolution>1</resolution>
                             <min_angle>${-fov/2}</min_angle>
@@ -135,5 +135,5 @@
                     </scan>
                     <range>
-                        <min>0.02</min>
+                        <min>0.01</min>
                         <max>${max_range}</max>
                         <resolution>0.01</resolution>
@@ -159,6 +159,8 @@
     <xacro:gazebo_ultrasonic name="us_top_left"   max_range="1.0" fov="0.2618"/>
     <xacro:gazebo_ultrasonic name="us_top_right"  max_range="1.0" fov="0.2618"/>
-    <xacro:gazebo_ultrasonic name="us_mid_left"   max_range="1.0" fov="0.2618"/>
-    <xacro:gazebo_ultrasonic name="us_mid_right"  max_range="1.0" fov="0.2618"/>
+    <xacro:gazebo_ultrasonic name="us_mid_1_left"   max_range="1.0" fov="0.2618"/>
+    <xacro:gazebo_ultrasonic name="us_mid_1_right"  max_range="1.0" fov="0.2618"/>
+    <xacro:gazebo_ultrasonic name="us_mid_2_left"   max_range="1.0" fov="0.2618"/>
+    <xacro:gazebo_ultrasonic name="us_mid_2_right"  max_range="1.0" fov="0.2618"/>
     <xacro:gazebo_ultrasonic name="us_bot_left"   max_range="1.0" fov="0.2618"/>
     <xacro:gazebo_ultrasonic name="us_bot_right"  max_range="1.0" fov="0.2618"/>

File: urdf/mobile_robot_v3.urdf.xacro (robot description, xacro)
@@ -41,5 +41,5 @@
         </inertial>
     </xacro:macro>
-    <xacro:include filename="gazebo_control_v2.xacro" />
+    <xacro:include filename="gazebo_control_v3.xacro" />
     <!-- ==================== PROPERTIES ==================== -->
     <xacro:property name="chassis_length" value="0.38"/>
@@ -166,9 +166,9 @@
         <parent link="chassis"/>
         <child link="laser_frame"/>
-        <origin xyz="0.257 0 0.075" rpy="0 0 0"/>
+        <origin xyz="0.257 0 0.075" rpy="0 0 3.14159"/>
     </joint>
     <link name="laser_frame">
         <visual>
-            <origin xyz="0 0 0" rpy="0 0 0"/>
+            <origin xyz="0 0 0" rpy="0 0 3.14159"/>
             <geometry>
                 <!-- <cylinder length="0.04" radius="0.038"/> -->
@@ -178,8 +178,8 @@
         </visual>
         <collision>
-            <origin xyz="0 0 0" rpy="0 0 0"/>
-            <geometry>
-                <!-- <cylinder length="0.04" radius="0.038"/> -->
-                <mesh filename="package://mobile_robot/meshes/RPLiDAR_s2.stl" scale="0.001 0.001 0.001"/>
+            <origin xyz="0 0 0" rpy="0 0 3.14159"/>
+            <geometry>
+                <cylinder length="0.04" radius="0.038"/>
+                <!-- <mesh filename="package://mobile_robot/meshes/RPLiDAR_s2.stl" scale="0.001 0.001 0.001"/> -->
             </geometry>
         </collision>
@@ -211,11 +211,11 @@
         <link name="${name}_link">
             <visual>
-                <geometry><box size="0.015 0.04 0.02"/></geometry>
+                <geometry><box size="0.015 0.02 0.04"/></geometry>
                 <material name="blue"/>
             </visual>
             <collision>
-                <geometry><box size="0.015 0.04 0.02"/></geometry>
+                <geometry><box size="0.015 0.02 0.04"/></geometry>
             </collision>
-            <xacro:inertial_box mass="0.01" x="0.015" y="0.04" z="0.02">
+            <xacro:inertial_box mass="0.01" x="0.015" y="0.02" z="0.04">
                 <origin xyz="0 0 0" rpy="0 0 0"/>
             </xacro:inertial_box>
@@ -225,5 +225,5 @@
         <parent link="chassis"/>
         <child link="us_top_left_link"/>
-        <origin xyz="0.35 0.17 0.49" rpy="0 0.4363 0"/>
+        <origin xyz="0.35 0.17 0.48" rpy="0 0 0"/>
     </joint>
     <xacro:ultrasonic_link name="us_top_left"/>
@@ -231,23 +231,35 @@
         <parent link="chassis"/>
         <child link="us_top_right_link"/>
-        <origin xyz="0.35 -0.17 0.49" rpy="0 0.4363 0"/>
+        <origin xyz="0.35 -0.17 0.48" rpy="0 0 0"/>
     </joint>
     <xacro:ultrasonic_link name="us_top_right"/>
-    <joint name="us_mid_left_joint" type="fixed">
-        <parent link="chassis"/>
-        <child link="us_mid_left_link"/>
-        <origin xyz="0.35 0.17 0.257" rpy="0 -0.2618 0"/>
-    </joint>
-    <xacro:ultrasonic_link name="us_mid_left"/>
-    <joint name="us_mid_right_joint" type="fixed">
-        <parent link="chassis"/>
-        <child link="us_mid_right_link"/>
-        <origin xyz="0.35 -0.17 0.257" rpy="0 -0.2618 0"/>
-    </joint>
-    <xacro:ultrasonic_link name="us_mid_right"/>
+    <joint name="us_mid_1_left_joint" type="fixed">
+        <parent link="chassis"/>
+        <child link="us_mid_1_left_link"/>
+        <origin xyz="0.35 0.17 0.36" rpy="0 0 0"/>
+    </joint>
+    <xacro:ultrasonic_link name="us_mid_1_left"/>
+    <joint name="us_mid_1_right_joint" type="fixed">
+        <parent link="chassis"/>
+        <child link="us_mid_1_right_link"/>
+        <origin xyz="0.35 -0.17 0.36" rpy="0 0 0"/>
+    </joint>
+    <xacro:ultrasonic_link name="us_mid_1_right"/>
+    <joint name="us_mid_2_left_joint" type="fixed">
+        <parent link="chassis"/>
+        <child link="us_mid_2_left_link"/>
+        <origin xyz="0.35 0.17 0.24" rpy="0 0 0"/>
+    </joint>
+    <xacro:ultrasonic_link name="us_mid_2_left"/>
+    <joint name="us_mid_2_right_joint" type="fixed">
+        <parent link="chassis"/>
+        <child link="us_mid_2_right_link"/>
+        <origin xyz="0.35 -0.17 0.24" rpy="0 0 0"/>
+    </joint>
+    <xacro:ultrasonic_link name="us_mid_2_right"/>
     <joint name="us_bot_left_joint" type="fixed">
         <parent link="chassis"/>
         <child link="us_bot_left_link"/>
-        <origin xyz="0.35 0.17 0.03" rpy="0 0.2618 0"/>
+        <origin xyz="0.35 0.17 0.12" rpy="0 0 0"/>
     </joint>
     <xacro:ultrasonic_link name="us_bot_left"/>
@@ -255,5 +267,5 @@
         <parent link="chassis"/>
         <child link="us_bot_right_link"/>
-        <origin xyz="0.35 -0.17 0.03" rpy="0 0.2618 0"/>
+        <origin xyz="0.35 -0.17 0.12" rpy="0 0 0"/>
     </joint>
     <xacro:ultrasonic_link name="us_bot_right"/>
